Commit message: Move `urdf_path` into `config.h`

File: models/L5.urdf (robot description, URDF)
Before this commit: robot ultron_v1.1_aa, 8 links, 7 joints
Links:
- link base_link: mass 0.428 -> 0.42272; geometry collision mesh filename=package://meshes/L5/base_link.STL; visual mesh filename=package://meshes/L5/base_link.STL
- link link1: mass 0.064 -> 0.09728; geometry collision mesh filename=package://meshes/L5/link1.STL; visual mesh filename=package://meshes/L5/link1.STL
- link link2: mass 1.165 -> 1.1477; geometry collision mesh filename=package://meshes/L5/link2.STL; visual mesh filename=package://meshes/L5/link2.STL
- link link3: mass 0.546 -> 0.66; geometry collision mesh filename=package://meshes/L5/link3.STL; visual mesh filename=package://meshes/L5/link3.STL
- link link4: mass 0.080971 -> 0.11714; geometry collision mesh filename=package://meshes/L5/link4.STL; visual mesh filename=package://meshes/L5/link4.STL
- link link5: mass 0.655 -> 0.6353; geometry collision mesh filename=package://meshes/L5/link5.STL; visual mesh filename=package://meshes/L5/link5.STL
- link link6: geometry collision mesh filename=package://meshes/L5/link6.STL; visual mesh filename=package://meshes/L5/link6.STL
Joints:
- joint gripper_fixed_joint: origin xyz=0.145 0.0 0.0 rpy=0 0 0 -> xyz=0.1576 0.0 0.0 rpy=0 0 0
- joint joint1: origin xyz=0 0 0.0603 rpy=0 0 0 -> xyz=0 0 0.0565 rpy=0 0 0
- joint joint2: limit lower=0 upper=3.14 effort=100 velocity=1000 -> lower=-10 upper=10 effort=100 velocity=1000; origin xyz=0.02 0 0.0402 rpy=0 0 0 -> xyz=0.02 0 0.047 rpy=0 0 0
- joint joint3: limit lower=0 upper=3.14 effort=30 velocity=10 -> lower=-10 upper=10 effort=100 velocity=1000; origin xyz=-0.264 0 0 rpy=-3.1416 0 0 -> xyz=-0.264 0 0 rpy=3.1416 0 0
- joint joint4: limit lower=-1.57079632679 upper=1.57079632679 effort=30 velocity=10 -> lower=-10 upper=10 effort=100 velocity=1000; origin xyz=0.245 0 -0.056 rpy=0 0 0 -> xyz=0.245 0 -0.06 rpy=0 0 0
- joint joint5: limit lower=-1.67 upper=1.67 effort=100 velocity=1000 -> lower=-10 upper=10 effort=100 velocity=1000; origin xyz=0.06575 -0.001 -0.0825 rpy=0 0 0 -> xyz=0.06775 -5E-05 -0.0865 rpy=0 0 0
- joint joint6: limit lower=-1.57 upper=1.57 effort=100 velocity=1000 -> lower=-10 upper=10 effort=100 velocity=1000; origin xyz=0.02845 0 0.0825 rpy=-3.1416 0 0 -> xyz=0.02895 0 0.0865 rpy=3.1416 0 0

File: models/X5.urdf (robot description, URDF)
Before this commit: robot arx5_gopro, 8 links, 7 joints
Links:
- link eef_link: mass 0.0001 -> 0.0
- link link1: geometry collision mesh filename=./meshes/X5/link1.STL; visual mesh filename=./meshes/X5/link1.STL
- link link2: geometry collision mesh filename=./meshes/X5/link2.STL; visual mesh filename=./meshes/X5/link2.STL
- link link3: geometry collision cylinder length=0.15 radius=0.02; visual mesh filename=./meshes/X5/link3.STL
- link link4: geometry collision cylinder length=0.05 radius=0.025; visual mesh filename=./meshes/X5/link4.STL
- link link5: geometry collision cylinder length=0.025 radius=0.02; visual mesh filename=./meshes/X5/link5.STL
- link link6: mass 0.902 -> 0.581000; geometry collision mesh filename=./meshes/X5/link6.STL; visual mesh filename=./meshes/X5/link6.STL
Joints:
- joint gripper_fixed_joint: origin xyz=0.225 0.0 0.0 rpy=0 0 0 -> xyz=0.145 0.0 0.0 rpy=0 0 0
- joint joint6: limit lower=-1.57 upper=1.57 effort=30 velocity=10 -> lower=-1.57 upper=1.57 effort=100 velocity=1000

Commit message: Update readme and L5 urdf

File: models/L5.urdf (robot description, URDF)
Before this commit: robot L5, 8 links, 7 joints
Joints:
- joint gripper_fixed_joint: origin xyz=0.1576 0.0 0.0 rpy=0 0 0 -> xyz=0.155 0.0 0.0 rpy=0 0 0

File: models/L5_umi.urdf (robot description, URDF)
Before this commit: robot L5_umi, 8 links, 7 joints
Joints:
- joint gripper_fixed_joint: origin xyz=0.2376 0.0 0.0 rpy=0 0 0 -> xyz=0.235 0.0 0.0 rpy=0 0 0
